File: keyboard-square-test/keyboard-square-test.kicad_sch (KiCad schematic)
At the start: 16 parts, among them SW1 SW_Push, U1 ATMEGA32U4-AU, Y1 16Mhz

Commit message: going well, really glad everything is well documented, though I don't think it's 100% complete but I'm figuring it out... Slowly...
Parts:
- added D1, D2, D3, D4: D_Small, Diode_SMD:D_SOD-123, symbol Device:D_Small
- added MX1, MX2, MX3, MX4: MX-NoLED, symbol MX_Alps_Hybrid:MX-NoLED
- C1, C2, C3, C4, C5, C6, C7: footprint (none) -> Capacitor_SMD:C_0805_2012Metric
- F1: footprint (none) -> Fuse:Fuse_1206_3216Metric
Connections:
- net D+: now also USB1.3 (D+)
- net D-: now also USB1.4 (D-)
- net GND: now also USB1.1 (GND)
- net at USB1.5 (VBUS): now also F1.1
- net VCC: no longer names the net of USB1.6 (SHIELD)
- net VCC: no longer F1.1
- new net: D4.2 (A), MX4.2 (ROW)
- new net: D2.2 (A), MX2.2 (ROW)
- new net: D1.2 (A), MX1.2 (ROW)
- new net: D3.2 (A), MX3.2 (ROW)
- new net COL0: MX1.1 (COL), MX3.1 (COL)
- new net COL1: MX2.1 (COL), MX4.1 (COL)
- new net ROW0: D1.1 (K), D2.1 (K)
- new net ROW1: D3.1 (K), D4.1 (K)
Other:
- moved on the sheet: C1, C2, C3, C4, C5, C6, C7, F1, R1, R2, R3, R4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
